Commit message: wip, actual status of raspberry dont merge

File: sar_description/urdf/control/ros2_control.urdf.xacro (robot description, xacro)
@@ -17,28 +17,20 @@
         <command_interface name="velocity" />
         <state_interface name="velocity" />
-        <xacro:if value="${use_sim}">
-          <state_interface name="position" />
-        </xacro:if>
+        <state_interface name="position" />
       </joint>
       <joint name="fr_wheel_joint">
         <command_interface name="velocity" />
         <state_interface name="velocity" />
-        <xacro:if value="${use_sim}">
-          <state_interface name="position" />
-        </xacro:if>
+        <state_interface name="position" />
       </joint>
       <joint name="rl_wheel_joint">
         <command_interface name="velocity" />
         <state_interface name="velocity" />
-        <xacro:if value="${use_sim}">
-          <state_interface name="position" />
-        </xacro:if>
+        <state_interface name="position" />
       </joint>
       <joint name="rr_wheel_joint">
         <command_interface name="velocity" />
         <state_interface name="velocity" />
-        <xacro:if value="${use_sim}">
-          <state_interface name="position" />
-        </xacro:if>
+        <state_interface name="position" />
       </joint>
     </ros2_control>

File: sar_description/urdf/sensors/rplidar.urdf.xacro (robot description, xacro)
@@ -5,5 +5,5 @@
       <parent link="body_link" />
       <child link="laser_frame" />
-      <origin xyz="${x} ${y} ${z}" rpy="0.0 0.0 0.0" />
+      <origin xyz="${x} ${y} ${z}" rpy="${pi} ${pi} 0.0" />
     </joint>
     <link name="laser_frame">
